Commit message: Updated arm.xacro

File: urdf/arm.xacro (robot description, xacro)
@@ -24,5 +24,5 @@
             <origin xyz="0 0 ${arm_base_height / 2.0}" rpy="0 0 0" />
         </collision>
-        <inertial>
+        <!-- <inertial>
             <origin xyz= "0 0 ${arm_base_height / 2.0}" rpy= "0 0 0"/>
             <mass value= "0.5" />
@@ -30,5 +30,7 @@
                      iyy = "${(0.5/12) * (arm_base_length * arm_base_length + arm_base_width * arm_base_width)}" iyz="0"
                      izz="${(0.5/12) * (arm_base_height * arm_base_height + arm_base_width * arm_base_width)}" />
-        </inertial>
+        </inertial> -->
+        <xacro:box_inertia m="0.5" l="${arm_base_length}" w="${arm_base_width}"
+        h="${arm_base_height}" xyz="0 0 ${arm_base_height/2.0}" rpy="0 0 0"/>
     </link>
     <link name="forearm_link">
@@ -48,5 +50,5 @@
             <origin xyz="0 0 ${forearm_length / 2.0}" rpy="0 0 0" />
         </collision>
-        <inertial>
+        <!-- <inertial>
             <origin xyz= "0 0 ${forearm_length / 2.0}" rpy= "0 0 0"/>
             <mass value= "0.3" />
@@ -54,5 +56,7 @@
                      iyy = "${(0.3/12) * (3 * forearm_radius * forearm_radius + forearm_length * forearm_length)}" iyz="0"
                      izz="${(0.3/2) * (forearm_radius * forearm_radius)}" />
-        </inertial>
+        </inertial> -->
+        <xacro:solid-cylinder_inertia m= "0.3" r= "${forearm_radius}"  h="${forearm_length}"
+                         xyz="0 0 ${forearm_length / 2.0}" rpy="0 0 0"/>
     </link>
     <link name="hand_link">
@@ -70,5 +74,5 @@
             <origin xyz="0 0 ${hand_length / 2.0}" rpy="0 0 0" />
         </collision>
-        <inertial>
+        <!-- <inertial>
             <origin xyz= "0 0 ${hand_length / 2.0}" rpy= "0 0 0"/>
             <mass value= "0.3" />
@@ -76,5 +80,7 @@
                      iyy = "${(0.3/12) * (3 * hand_radius * hand_radius + hand_length * hand_length)}" iyz="0"
                      izz="${(0.3/2) * (hand_radius * hand_radius)}" />
-        </inertial>
+        </inertial> -->
+        <xacro:solid-cylinder_inertia m= "0.3" r= "${hand_radius}"  h="${hand_length}"
+            xyz="0 0 ${hand_length / 2.0}" rpy="0 0 0"/>
     </link>
     <joint name="arm_base_forearm_joint" type="revolute">
